Commit message: Odometry node created and not working

File: sagan_description/model/Sagan.xacro.urdf (robot description, URDF)
Before this commit: robot Sagan, 12 links, 11 joints
Links:
- added link odom
Joints:
- added joint odom_to_base_footprint: type fixed, parent odom, child base_footprint, origin xyz=0 0 0 rpy=0 0 0

Commit message: wheel interface congigured to effort

File: sagan_description/model/Sagan.xacro.urdf (robot description, URDF)
Before this commit: robot Sagan, 13 links, 12 joints
Links:
- added link world
Joints:
- added joint world_to_odom: type fixed, parent world, child odom, origin xyz=0 0 0 rpy=0 0 0

File: sagan_description/model/ros2_control.xacro (robot description, xacro)
@@ -11,4 +11,5 @@
             </command_interface>
             <command_interface name="position" />
+            <command_interface name="effort" />
             <state_interface name="velocity" />
             <state_interface name="position"/>
@@ -20,4 +21,5 @@
             </command_interface>
             <command_interface name="position" />
+            <command_interface name="effort" />
             <state_interface name="velocity" />
             <state_interface name="position"/>
@@ -29,4 +31,5 @@
             </command_interface>
             <command_interface name="position" />
+            <command_interface name="effort" />
             <state_interface name="velocity" />
             <state_interface name="position"/>
@@ -38,4 +41,5 @@
             </command_interface>
             <command_interface name="position" />
+            <command_interface name="effort" />
             <state_interface name="velocity" />
             <state_interface name="position"/>

Commit message: wheel emulator added

File: sagan_description/model/Sagan.xacro.urdf (robot description, URDF)
Before this commit: robot Sagan, 14 links, 13 joints
Joints:
- joint world_to_odom: origin xyz=0 0 0 rpy=0 0 0 -> xyz=0 0 1 rpy=0 0 0

File: sagan_description/model/ros2_control.xacro (robot description, xacro)
@@ -58,4 +58,5 @@
                 <param name="max">90</param>
             </command_interface>
+            <command_interface name="effort" />
             <state_interface name="velocity" />
             <state_interface name="position"/>
@@ -71,4 +72,5 @@
                 <param name="max">90</param>
             </command_interface>
+            <command_interface name="effort" />
             <state_interface name="velocity" />
             <state_interface name="position"/>
@@ -84,4 +86,5 @@
                 <param name="max">90</param>
             </command_interface>
+            <command_interface name="effort" />
             <state_interface name="velocity" />
             <state_interface name="position"/>
@@ -97,4 +100,5 @@
                 <param name="max">90</param>
             </command_interface>
+            <command_interface name="effort" />
             <state_interface name="velocity" />
             <state_interface name="position"/>]

Commit message: Steering emulator actualized

File: sagan_description/model/Sagan.xacro.urdf (robot description, URDF)
Before this commit: robot Sagan, 14 links, 13 joints
Links:
- removed link world
Joints:
- removed joint world_to_odom

Commit message: Imu sensor added and not working properly

File: sagan_description/model/Sagan.xacro.urdf (robot description, URDF)
Before this commit: robot Sagan, 13 links, 12 joints
Links:
- added link imu_link, mass 0
Joints:
- added joint imu_joint: type fixed, parent base_link, child imu_link, origin xyz=0 0 0 rpy=0 0 0, axis 0 0.1 0

Commit message: efk added

File: sagan_description/model/Sagan.xacro.urdf (robot description, URDF)
Before this commit: robot Sagan, 14 links, 13 joints
Links:
- added link efk_reference
- added link gz_reference
- added link odom_gz_link, mass 0
Joints:
- added joint odom_efk_joint: type fixed, parent odom, child efk_reference, origin xyz=0 0 0 rpy=0 0 0
- added joint odom_gz_joint: type fixed, parent base_link, child odom_gz_link, origin xyz=0 0 0 rpy=-1.5708 0 0, axis 0 0 0
- added joint odom_gz_reference_joint: type fixed, parent odom, child gz_reference
- joint imu_joint: axis 0 0.1 0 -> 0 0 0; origin xyz=0 0 0 rpy=0 0 0 -> xyz=0 0 0 rpy=-1.5708 0 0

Commit message: Sagan URDF colision model of the wheel changed

File: sagan_description/model/Sagan.xacro.urdf (robot description, URDF)
Before this commit: robot Sagan, 17 links, 16 joints
Links:
- link LF_stering_arm: mass 0.457316704111482 -> 0.457
- link LF_wheel: mass 0.504199735680765 -> 0.500; geometry collision cylinder length=0.06 radius=0.06; visual mesh filename=file://$(find sagan_description)/model/meshes/LF_wheel.STL
- link LR_stering_arm: mass 0.457316671284394 -> 0.457
- link LR_wheel: mass 0.504199729718972 -> 0.500; geometry collision cylinder length=0.06 radius=0.06; visual mesh filename=file://$(find sagan_description)/model/meshes/LR_wheel.STL
- link RF_stering_arm: mass 0.457316670820617 -> 0.457
- link RF_wheel: mass 0.504199732627693 -> 0.500; geometry collision cylinder length=0.06 radius=0.06; visual mesh filename=file://$(find sagan_description)/model/meshes/RF_wheel.STL
- link RR_stering_arm: mass 0.457316705822729 -> 0.457
- link RR_wheel: mass 0.504199733126219 -> 0.500; geometry collision cylinder length=0.06 radius=0.06; visual mesh filename=file://$(find sagan_description)/model/meshes/RR_wheel.STL
Joints:
- joint imu_joint: origin xyz=0 0 0 rpy=-1.5708 0 0 -> xyz=0 0 0 rpy=-1.5708 0 3.1415

Commit message: Robot URDF modified

File: sagan_description/model/Sagan.xacro.urdf (robot description, URDF)
Before this commit: robot Sagan, 17 links, 16 joints
Links:
- link LF_stering_arm: geometry visual mesh filename=file://$(find sagan_description)/model/meshes/LF_stering_ar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
- link LF_wheel: geometry collision cylinder length=0.01 radius=0.06; visual mesh filename=file://$(find sagan_description)/model/meshes/LF_wheel.STL
- link LR_stering_arm: geometry visual mesh filename=file://$(find sagan_description)/model/meshes/LR_stering_ar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
- link LR_wheel: geometry collision cylinder length=0.01 radius=0.06; visual mesh filename=file://$(find sagan_description)/model/meshes/LR_wheel.STL
- link Left_arm: mass 0.351441910668664 -> 0.3514
- link RF_stering_arm: geometry visual mesh filename=file://$(find sagan_description)/model/meshes/RF_stering_ar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
- link RF_wheel: geometry collision cylinder length=0.01 radius=0.06; visual mesh filename=file://$(find sagan_description)/model/meshes/RF_wheel.STL
- link RR_stering_arm: geometry visual mesh filename=file://$(find sagan_description)/model/meshes/RR_stering_ar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
- link RR_wheel: geometry collision cylinder length=0.01 radius=0.06; visual mesh filename=file://$(find sagan_description)/model/meshes/RR_wheel.STL
- link base_link: mass 1.64102297043224 -> ${m_base}

Commit message: URDF modified

File: sagan_description/model/Sagan.xacro.urdf (robot description, URDF)
Before this commit: robot Sagan, 17 links, 16 joints
Links:
- link LF_stering_arm: mass 0.457 -> ${m_steering_arm}
- link LF_wheel: mass 0.500 -> ${m_wheel}
- link LR_stering_arm: mass 0.457 -> ${m_steering_arm}
- link LR_wheel: mass 0.500 -> ${m_wheel}
- link Left_arm: mass 0.3514 -> ${m_arm}
- link RF_stering_arm: mass 0.457 -> ${m_steering_arm}
- link RF_wheel: mass 0.500 -> ${m_wheel}
- link RR_stering_arm: mass 0.457 -> ${m_steering_arm}
- link RR_wheel: mass 0.500 -> ${m_wheel}
- link Right_arm: mass 0.351441923670602 -> ${m_arm}

Commit message: Sagan no rviz e gazebo, porém rotacionado no rviz

File: sagan_description/model/Sagan.xacro.urdf (robot description, URDF)
Before this commit: robot Sagan, 17 links, 16 joints
Joints:
- joint odom_gz_joint: origin xyz=0 0 0 rpy=-1.5708 0 0 -> xyz=0 0 0 rpy=0 0 0

Commit message: friction coefficients and URDF settings modified

File: sagan_description/model/Sagan.xacro.urdf (robot description, URDF)
Before this commit: robot Sagan, 17 links, 16 joints
Links:
- link LF_wheel: geometry collision sphere radius=0.06; visual mesh filename=file://$(find sagan_description)/model/meshes/LF_wheel.STL
- link LR_wheel: geometry collision sphere radius=0.06; visual mesh filename=file://$(find sagan_description)/model/meshes/LR_wheel.STL
- link RF_wheel: geometry collision sphere radius=0.06; visual mesh filename=file://$(find sagan_description)/model/meshes/RF_wheel.STL
- link RR_wheel: geometry collision sphere radius=0.06; visual mesh filename=file://$(find sagan_description)/model/meshes/RR_wheel.STL

Commit message: friction coefficient modified

File: sagan_description/model/Sagan.xacro.urdf (robot description, URDF)
Before this commit: robot Sagan, 17 links, 16 joints
Joints:
- joint odom_gz_joint: origin xyz=0 0 0 rpy=-1.5708 0 0 -> xyz=0 0 0 rpy=-1.5707963268 0 0

Commit message: Kalman filter and odometry package modified

File: sagan_description/model/Sagan.xacro.urdf (robot description, URDF)
Before this commit: robot Sagan, 17 links, 16 joints
Links:
- added link noise_odometry
Joints:
- added joint odom_noise_joint: type fixed, parent odom, child noise_odometry, origin xyz=0 0 0 rpy=0 0 0

Commit message: working slam

File: sagan_description/model/Sagan.xacro.urdf (robot description, URDF)
Before this commit: robot Sagan, 18 links, 17 joints
Links:
- added link lidar_link, mass 1e-6; collision cylinder length=0.1 radius=0.1; visual cylinder length=0.02 radius=0.03
Joints:
- added joint lidar_joint: type fixed, parent base_link, child lidar_link, origin xyz=-0.03 -0.095 0 rpy=1.5707 0 0, axis 0 0 1
